File: MATRIX.sch (KiCad schematic (older format))
At the start: 95 parts

Commit message: Finished routing, SS
Parts:
- removed D? (x5): D, Keebio-Parts:Diode, symbol device:D_ALT
- removed MX?: MX-ISO, MX_Alps_Hybrid:MX-ISO-ReversedStabilizers, symbol MX_Alps_Hybrids:MX-ISO
- removed MX?: MX-6.25U, MX_Alps_Hybrid:MX-6.25U, symbol MX_Alps_Hybrids:MX-6.25U
- removed MX?: MX-1.75U, MX_Alps_Hybrid:MX-1.75U, symbol MX_Alps_Hybrids:MX-1.75U
- removed MX?: MX-2.25U, MX_Alps_Hybrid:MX-2.25U, symbol MX_Alps_Hybrids:MX-2.25U
- removed MX? (x2): MX-1.25U, symbol MX_Alps_Hybrids:MX-1.25U
- added D42, D43, D44, D45, D46, D47, D48, D49, D50, D51, D52, D53, D54, D55, D57, D58, D59, D60, D61, D62: D, Diode_SMD:D_SOD-123, symbol device:D_ALT
- added MX29, MX43: MX-1.25U, keyboard_parts:ALPS_PLATE_SPRING_1.25U, symbol MX_Alps_Hybrids:MX-1.25U
- added MX44, MX45, MX46, MX47, MX48, MX49, MX50, MX51, MX52, MX53, MX54, MX56, MX59, MX63: MX-1U, keyboard_parts:ALPS_PLATE_SPRING, symbol MX_Alps_Hybrids:MX-1U
- added MX55: MX-1.75U, keyboard_parts:ALPS_PLATE_SPRING_1.75U, symbol MX_Alps_Hybrids:MX-1.75U
- added MX57: MX-2.75U, keyboard_parts:ALPS_PLATE_SPRING2.75U, symbol MX_Alps_Hybrids:MX-2.75U
- added MX60, MX62, MX64: MX-1.5U, keyboard_parts:ALPS_PLATE_SPRING1.5U, symbol MX_Alps_Hybrids:MX-1.5U
- added MX61: MX-7U, keyboard_parts:ALPS_PLATE_SPRING7U, symbol MX_Alps_Hybrids:MX-7U
- D1: footprint Keebio-Parts:Diode -> Diode_SMD:D_SOD-123
- D10, D11, D12, D13, D14, D15, D16, D17, D18, D19, D2, D20, D21, D22, D23, D24, D25, D26, D27, D28, D29, D3, D30, D31, D32, D33, D34, D35, D36, D37, D38, D39, D4, D40, D41, D5, D56, D6, D7, D8, D9: renamed from D?; footprint Keebio-Parts:Diode -> Diode_SMD:D_SOD-123
- MX1: footprint MX_Alps_Hybrid:MX-1U -> keyboard_parts:ALPS_PLATE_SPRING
- MX10, MX11, MX12, MX13, MX16, MX17, MX18, MX19, MX2, MX20, MX21, MX22, MX23, MX24, MX25, MX26, MX27, MX3, MX31, MX32, MX33, MX34, MX35, MX36, MX37, MX38, MX39, MX4, MX40, MX41, MX42, MX5, MX6, MX7, MX8, MX9: renamed from MX?; footprint MX_Alps_Hybrid:MX-1U -> keyboard_parts:ALPS_PLATE_SPRING
- MX14: renamed from MX?; footprint (none) -> keyboard_parts:ALPS_PLATE_SPRING2U
- MX15, MX58: renamed from MX?; footprint MX_Alps_Hybrid:MX-1.5U -> keyboard_parts:ALPS_PLATE_SPRING1.5U
- MX28: renamed from MX?; footprint MX_Alps_Hybrid:MX-ISO-ReversedStabilizers -> keyboard_parts:ALPS_PLATE_SPRINGISOCOMBINED
- MX30: renamed from MX?; footprint MX_Alps_Hybrid:MX-1.75U -> keyboard_parts:ALPS_PLATE_SPRING_1.75U
Connections:
- net labels added: C0, C1, C10, C11, C12, C13, C2, C3, C4, C5, C6, C7, C8, C9, R0, R1, R2, R3, R4
- wire segments 47 -> 192
Other:
- moved on the sheet: D56, MX58
