File: PROJECT.sch (KiCad schematic (older format))
At the start: 21 parts, among them J1 USB_mini_micro_B, SW1 SW_PUSH, U1 PRTR5V0U2X, U2 ATmega32U4, X1 XTAL_GND

Commit message: Finished routing, SS
Parts:
- C1, C2, C3, C4, C5, C6, C7, C8, USBCap1: footprint (none) -> Capacitor_SMD:C_0805_2012Metric_Pad1.15x1.40mm_HandSolder
- F1: footprint (none) -> Fuse:Fuse_0805_2012Metric_Pad1.15x1.40mm_HandSolder
- J1: footprint (none) -> Mixed Lib:USB
- R1, R2, UR1, UR2, UR5: footprint (none) -> Resistor_SMD:R_0805_2012Metric_Pad1.15x1.40mm_HandSolder
- SPI1: footprint (none) -> keyboard_parts:Pin_Header_Straight_2x03_Pitch2.00mm; symbol conn:Conn_02x03_Counter_Clockwise -> PROJECT-rescue:Conn_02x03_Counter_Clockwise-conn
- SW1: footprint (none) -> Button_Switch_SMD:SW_SPST_SKQG_WithStem
- U1: footprint (none) -> Mixed Lib:SOT143B
- U2: footprint (none) -> keyboard_parts:QFP44; symbol atmel:ATmega32U4 -> PROJECT-rescue:ATmega32U4-atmel
- X1: footprint (none) -> keyboard_parts:Crystal_SMD_3225-4pin_3.2x2.5mm
Connections:
- net labels added: C0, C1, C10, C11, C12, C13, C2, C3, C4, C5, C6, C7, C8, C9, R0, R1, R2, R3, R4
- wire segments 83 -> 94
